File: RcCtlHw.kicad_pcb (KiCad board)
At the start: 2 copper layers, 26.7 x 41.9 mm, 30 parts, among them J1 USB_B_Mini, J2 Program, J3 TFT_LCD, SW1 On/Off, U1 TP4056, U2 ESP-M2, U3 ADS1015, U4 Joystick

Commit message: Move switch to before regulator
Parts:
- moved C4 2.00 mm to (136.9, 121.7), turned to 180 degrees
- moved C3 1.19 mm to (136.9, 119.5), turned to 180 degrees
- turned C8 to 180 degrees
Connections:
- C3 pad 1: Net-(C3-Pad1) -> +3V3
- C4 pad 1: Net-(C3-Pad1) -> +3V3
- SW1 pad 1: Net-(C3-Pad1) -> +BATT
- SW1 pad 2: +3V3 -> Net-(SW1-Pad2)
- V1 pad 1: +BATT -> Net-(SW1-Pad2)
- V1 pad 3: Net-(C3-Pad1) -> +3V3
Routing:
- net Net-(C3-Pad1): track 23.1 -> 0.00 mm, vias 1 -> 0
- net +3V3: track 154.5 -> 172.5 mm
- net Net-(SW1-Pad2): track 0.00 -> 13.2 mm, vias 0 -> 1
- net +BATT: track 85.2 -> 81.2 mm
- net Net-(C8-Pad1): track 57.2 -> 55.1 mm
- net GND: track 154.4 -> 156.4 mm, vias 3 -> 4
- net Net-(C1-Pad1): track 24.5 -> 23.7 mm
- net /TFT_SDA: track 30.3 -> 29.8 mm
